File: pcb/keyboard.kicad_pcb (KiCad board)
At the start: 2 copper layers, 349.9 x 134.6 mm, 170 parts, among them SW1 SW_Push, SW10 SW_Push, SW11 SW_Push, SW12 SW_Push, SW13 SW_Push, SW14 SW_Push, SW15 SW_Push, SW16 SW_Push, SW17 SW_Push, SW18 SW_Push, SW19 SW_Push, SW2 SW_Push, SW20 SW_Push, SW21 SW_Push, SW22 SW_Push, SW23 SW_Push, SW24 SW_Push, SW25 SW_Push, SW26 SW_Push, SW27 SW_Push, SW28 SW_Push, SW29 SW_Push, SW3 SW_Push, SW30 SW_Push, SW31 SW_Push, SW32 SW_Push, SW33 SW_Push, SW34 SW_Push, SW35 SW_Push, SW36 SW_Push, SW37 SW_Push, SW38 SW_Push, SW39 SW_Push, SW4 SW_Push, SW40 SW_Push, SW41 SW_Push, SW42 SW_Push, SW43 SW_Push, SW44 SW_Push, SW45 SW_Push, SW46 SW_Push, SW47 SW_Push, SW48 SW_Push, SW49 SW_Push, SW5 SW_Push, SW50 SW_Push, SW51 SW_Push, SW52 SW_Push, SW53 SW_Push, SW54 SW_Push, SW55 SW_Push, SW56 SW_Push, SW57 SW_Push, SW58 SW_Push, SW59 SW_Push, SW6 SW_Push, SW60 SW_Push, SW61 SW_Push, SW62 SW_Push, SW63 SW_Push, SW64 SW_Push, SW65 SW_Push, SW66 SW_Push, SW67 SW_Push, SW68 SW_Push, SW69 SW_Push, SW7 SW_Push, SW70 SW_Push, SW71 SW_Push, SW72 SW_Push, SW73 SW_Push, SW74 SW_Push, SW75 SW_Push, SW76 SW_Push, SW77 SW_Push, SW78 SW_Push, SW79 SW_Push, SW8 SW_Push, SW80 SW_Push, SW81 SW_Push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

Commit message: Add files via upload
Parts:
- SW50, SW51: footprint Button_Switch_Keyboard:SW_Cherry_MX_1.00u_PCB -> Button_Switch_Keyboard:SW_Cherry_MX_1.75u_PCB
- SW59: footprint Button_Switch_Keyboard:SW_Cherry_MX_1.00u_PCB -> Button_Switch_Keyboard:SW_Cherry_MX_2.75u_PCB
- moved SW50 7.14 mm to (194.5, -153.7)
- moved SW51 7.14 mm to (194.5, -134.6)
Routing:
- net Net-(D32-A): track 5.85 -> 13.0 mm
- net Column 11: track 660.2 -> 660.5 mm, vias 13 -> 14
Other:
- outline, holes or cut-outs redrawn
Changed lines of the file:
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@@
 		)
 	)
-	(footprint "Button_Switch_Keyboard:SW_Cherry_MX_1.00u_PCB"
+	(footprint "Button_Switch_Keyboard:SW_Cherry_MX_2.75u_PCB"
 		(layer "F.Cu")
 		(at 311.15 -115.57)
-		(descr "Cherry MX keyswitch, 1.00u, PCB mount, http://cherryamericas.com/wp-content/uploads/2014/12/mx_cat.pdf")
-		(tags "Cherry MX keyswitch 1.00u PCB")
+		(descr "Cherry MX keyswitch, 2.75u, PCB mount, http://cherryamericas.com/wp-content/uploads/2014/12/mx_cat.pdf")
+		(tags "Cherry MX keyswitch 2.75u PCB")
 		(property "Reference" "SW59"
 			(at -2.54 -2.794 0)
@@
 			)
 		)
-		(property "Footprint" "Button_Switch_Keyboard:SW_Cherry_MX_1.00u_PCB"
+		(property "Footprint" "Button_Switch_Keyboard:SW_Cherry_MX_2.75u_PCB"
 			(at 0 0 0)
 			(unlocked yes)
@@
 		)
 		(fp_line
-			(start -12.065 -4.445)
-			(end 6.985 -4.445)
+			(start -28.73375 -4.445)
+			(end 23.65375 -4.445)
 			(stroke
 				(width 0.15)
@@
 		)
 		(fp_line
-			(start -12.065 14.605)
-			(end -12.065 -4.445)
+			(start -28.73375 14.605)
+			(end -28.73375 -4.445)
 			(stroke
 				(width 0.15)
@@
 		)
 		(fp_line
-			(start 6.985 -4.445)
-			(end 6.985 14.605)
+			(start 23.65375 -4.445)
+			(end 23.65375 14.605)
 			(stroke
 				(width 0.15)
@@
 		)
 		(fp_line
-			(start 6.985 14.605)
-			(end -12.065 14.605)
+			(start 23.65375 14.605)
+			(end -28.73375 14.605)
 			(stroke
 				(width 0.15)
@@
 		)
 		(pad "" np_thru_hole circle
+			(at -14.44 -1.92)
+			(size 3.05 3.05)
+			(drill 3.05)
+			(layers "*.Cu" "*.Mask")
+		)
+		(pad "" np_thru_hole circle
+			(at -14.44 13.32)
+			(size 4 4)
+			(drill 4)
+			(layers "*.Cu" "*.Mask")
+		)
+		(pad "" np_thru_hole circle
 			(at -7.62 5.08)
 			(size 1.7 1.7)
@@
 			(layers "*.Cu" "*.Mask")
 		)
+		(pad "" np_thru_hole circle
+			(at 9.36 -1.92)
+			(size 3.05 3.05)
+			(drill 3.05)
+			(layers "*.Cu" "*.Mask")
+		)
+		(pad "" np_thru_hole circle
+			(at 9.36 13.32)
+			(size 4 4)
+			(drill 4)
+			(layers "*.Cu" "*.Mask")
+		)
 		(pad "1" thru_hole circle
 			(at 0 0)
@@
 			(pintype "passive")
 		)
-		(model "${KICAD8_3DMODEL_DIR}/Button_Switch_Keyboard.3dshapes/SW_Cherry_MX_1.00u_PCB.wrl"
+		(model "${KICAD8_3DMODEL_DIR}/Button_Switch_Keyboard.3dshapes/SW_Cherry_MX_2.75u_PCB.wrl"
 			(offset
 				(xyz 0 0 0)
@@
 		)
 	)
-	(footprint "Button_Switch_Keyboard:SW_Cherry_MX_1.00u_PCB"
+	(footprint "Button_Switch_Keyboard:SW_Cherry_MX_1.75u_PCB"
 		(layer "F.Cu")
-		(at 187.325 -153.67)
-		(descr "Cherry MX keyswitch, 1.00u, PCB mount, http://cherryamericas.com/wp-content/uploads/2014/12/mx_cat.pdf")
-		(tags "Cherry MX keyswitch 1.00u PCB")
+		(at 194.4624 -153.67)
+		(descr "Cherry MX keyswitch, 1.75u, PCB mount, http://cherryamericas.com/wp-content/uploads/2014/12/mx_cat.pdf")
+		(tags "Cherry MX keyswitch 1.75u PCB")
 		(property "Reference" "SW50"
 			(at -2.54 -2.794 0)
@@
 			)
 		)
-		(property "Footprint" "Button_Switch_Keyboard:SW_Cherry_MX_1.00u_PCB"
+		(property "Footprint" "Button_Switch_Keyboard:SW_Cherry_MX_1.75u_PCB"
 			(at 0 0 0)
 			(unlocked yes)
@@
 		)
 		(fp_line
-			(start -12.065 -4.445)
-			(end 6.985 -4.445)
+			(start -19.20875 -4.445)
+			(end 14.12875 -4.445)
 			(stroke
 				(width 0.15)
@@
 		)
 		(fp_line
-			(start -12.065 14.605)
-			(end -12.065 -4.445)
+			(start -19.20875 14.605)
+			(end -19.20875 -4.445)
 			(stroke
 				(width 0.15)
@@
 		)
 		(fp_line
-			(start 6.985 -4.445)
-			(end 6.985 14.605)
+			(start 14.12875 -4.445)
+			(end 14.12875 14.605)
 			(stroke
 				(width 0.15)
@@
 		)
 		(fp_line
-			(start 6.985 14.605)
-			(end -12.065 14.605)
+			(start 14.12875 14.605)
+			(end -19.20875 14.605)
 			(stroke
 				(width 0.15)
@@
 			(pintype "passive")
 		)
-		(model "${KICAD8_3DMODEL_DIR}/Button_Switch_Keyboard.3dshapes/SW_Cherry_MX_1.00u_PCB.wrl"
+		(model "${KICAD8_3DMODEL_DIR}/Button_Switch_Keyboard.3dshapes/SW_Cherry_MX_1.75u_PCB.wrl"
 			(offset
 				(xyz 0 0 0)
@@
 		)
 	)
-	(footprint "Button_Switch_Keyboard:SW_Cherry_MX_1.00u_PCB"
+	(footprint "Button_Switch_Keyboard:SW_Cherry_MX_1.75u_PCB"
 		(layer "F.Cu")
-		(at 187.325 -134.62)
-		(descr "Cherry MX keyswitch, 1.00u, PCB mount, http://cherryamericas.com/wp-content/uploads/2014/12/mx_cat.pdf")
-		(tags "Cherry MX keyswitch 1.00u PCB")
+		(at 194.4624 -134.62)
+		(descr "Cherry MX keyswitch, 1.75u, PCB mount, http://cherryamericas.com/wp-content/uploads/2014/12/mx_cat.pdf")
+		(tags "Cherry MX keyswitch 1.75u PCB")
 		(property "Reference" "SW51"
 			(at -2.54 -2.794 0)
@@
 			)
 		)
-		(property "Footprint" "Button_Switch_Keyboard:SW_Cherry_MX_1.00u_PCB"
+		(property "Footprint" "Button_Switch_Keyboard:SW_Cherry_MX_1.75u_PCB"
 			(at 0 0 0)
 			(unlocked yes)
@@
 		)
 		(fp_line
-			(start -12.065 -4.445)
-			(end 6.985 -4.445)
+			(start -19.20875 -4.445)
+			(end 14.12875 -4.445)
 			(stroke
 				(width 0.15)
@@
 		)
 		(fp_line
-			(start -12.065 14.605)
-			(end -12.065 -4.445)
+			(start -19.20875 14.605)
+			(end -19.20875 -4.445)
 			(stroke
 				(width 0.15)
@@
 		)
 		(fp_line
-			(start 6.985 -4.445)
-			(end 6.985 14.605)
+			(start 14.12875 -4.445)
+			(end 14.12875 14.605)
 			(stroke
 				(width 0.15)
@@
 		)
 		(fp_line
-			(start 6.985 14.605)
-			(end -12.065 14.605)
+			(start 14.12875 14.605)
+			(end -19.20875 14.605)
 			(stroke
 				(width 0.15)
@@
 			(pintype "passive")
 		)
-		(model "${KICAD8_3DMODEL_DIR}/Button_Switch_Keyboard.3dshapes/SW_Cherry_MX_1.00u_PCB.wrl"
+		(model "${KICAD8_3DMODEL_DIR}/Button_Switch_Keyboard.3dshapes/SW_Cherry_MX_1.75u_PCB.wrl"
 			(offset
 				(xyz 0 0 0)
@@
 	(gr_poly
 		(pts
-			(xy 523.875 -100.33) (xy 523.875 -218.44) (xy 413.385 -218.44) (xy 404.495 -234.95) (xy 346.075 -234.95)
-			(xy 336.55 -215.9) (xy 327.66 -196.85) (xy 270.51 -196.85) (xy 261.62 -215.9) (xy 184.15 -215.9)
-			(xy 173.99 -195.58) (xy 173.99 -100.33)
+			(xy 523.875 -99.695) (xy 523.875 -217.805) (xy 413.385 -217.805) (xy 404.495 -234.315) (xy 346.075 -234.315)
+			(xy 336.55 -215.265) (xy 327.66 -196.215) (xy 270.51 -196.215) (xy 261.62 -215.265) (xy 184.15 -215.265)
+			(xy 173.99 -194.945) (xy 173.99 -99.695)
 		)
 		(stroke
@@
 	)
 	(segment
-		(start 175.575 -132.08)
-		(end 175.26 -131.765)
+		(start 175.26 -131.765)
+		(end 175.575 -132.08)
 		(width 0.2)
 		(layer "F.Cu")
@@
 	)
 	(segment
-		(start 180.975 -132.08)
-		(end 175.575 -132.08)
+		(start 175.575 -132.08)
+		(end 188.1124 -132.08)
 		(width 0.2)
 		(layer "F.Cu")
@@
 	)
 	(segment
+		(start 191.135 -137.0838)
+		(end 191.135 -138.43)
+		(width 0.2)
+		(layer "F.Cu")
+		(net 114)
+	)
+	(segment
+		(start 192.7352 -136.3472)
+		(end 191.8716 -136.3472)
+		(width 0.2)
+		(layer "F.Cu")
+		(net 114)
+	)
+	(segment
 		(start 484 -137.03)
 		(end 484 -130.156598)
@@
 	)
 	(segment
+		(start 191.8716 -136.3472)
+		(end 191.135 -137.0838)
+		(width 0.2)
+		(layer "F.Cu")
+		(net 114)
+	)
+	(segment
 		(start 323.215 -174.625)
 		(end 321.31 -174.625)
@@
 	)
 	(segment
+		(start 194.4624 -134.62)
+		(end 192.7352 -136.3472)
+		(width 0.2)
+		(layer "F.Cu")
+		(net 114)
+	)
+	(segment
 		(start 443.865 -107.315)
 		(end 443.865 -107.95)
@@
 	)
 	(via
+		(at 191.135 -138.43)
+		(size 0.6)
+		(drill 0.3)
+		(layers "F.Cu" "B.Cu")
+		(net 114)
+	)
+	(via
 		(at 347.345 -163.195)
 		(size 0.6)
@@
 		(width 0.2)
 		(layer "B.Cu")
-		(net 114)
-	)
-	(segment
-		(start 187.325 -134.62)
-		(end 191.135 -138.43)
-		(width 0.2)
-		(layer "B.Cu")
